Commit message: lidarrr

File: description/robot.urdf.xacro (robot description, xacro)
@@ -3,3 +3,4 @@
     <xacro:include  filename="robot_core.xacro" />
     <xacro:include  filename="gazebo_control.xacro" />
+    <xacro:include  filename="lidar.xacro" />
 </robot>

File: description/robot_core.xacro (robot description, xacro)
@@ -10,4 +10,7 @@
     <material name="blue">
         <color rgba="0.2 0.2 1 1" />
+    </material>
+    <material name="red">
+        <color rgba="1 0 0 1" />
     </material>
     <material name="black">

Commit message: bugları düzelt

File: description/robot.urdf.xacro (robot description, xacro)
@@ -1,6 +1,11 @@
 <?xml version="1.0"?>
 <robot xmlns:xacro="http://www.ros.org/wiki/xacro"  name="robot">
-    <xacro:include  filename="ros2_control.xacro" />
-    <!-- <xacro:include  filename="gazebo_control.xacro" /> -->
+    <xacro:arg name="use_ros2_control" default="true"/>
+    <xacro:if value_"$(use_ros2_control)">
+        <xacro:include  filename="ros2_control.xacro" />
+    </xacro:if>
+    <xacro:unless value_"$(use_ros2_control)">
+        <xacro:include  filename="gazebo_control.xacro" />
+    </xacro:unless>
     <xacro:include  filename="robot_core.xacro" />
     <xacro:include  filename="lidar.xacro" />

File: description/robot_core.xacro (robot description, xacro)
@@ -63,5 +63,5 @@
         <collision>
             <geometry>
-                <cylinder radius="0.05" length="0.04"/>
+                <sphere radius="0.05"/>
             </geometry>
         </collision>
@@ -89,5 +89,5 @@
         <collision>
             <geometry>
-                <cylinder radius="0.05" length="0.04"/>
+                <sphere radius="0.05"/>
             </geometry>
         </collision>

Commit message: ahh ah

File: description/robot.urdf.xacro (robot description, xacro)
@@ -1,11 +1,6 @@
 <?xml version="1.0"?>
 <robot xmlns:xacro="http://www.ros.org/wiki/xacro"  name="robot">
-    <xacro:arg name="use_ros2_control" default="true"/>
-    <xacro:if value="$(arg use_ros2_control)">
-        <xacro:include filename="ros2_control.xacro" />
-    </xacro:if>
-    <xacro:unless value="$(arg use_ros2_control)">
-        <xacro:include filename="gazebo_control.xacro" />
-    </xacro:unless>
+    <xacro:include  filename="ros2_control.xacro" />
+    <!-- <xacro:include  filename="gazebo_control.xacro" /> -->
     <xacro:include  filename="robot_core.xacro" />
     <xacro:include  filename="lidar.xacro" />

File: description/robot_core.xacro (robot description, xacro)
@@ -63,5 +63,5 @@
         <collision>
             <geometry>
-                <sphere radius="0.05"/>
+                <cylinder radius="0.05" length="0.04"/>
             </geometry>
         </collision>
@@ -89,5 +89,5 @@
         <collision>
             <geometry>
-                <sphere radius="0.05"/>
+                <cylinder radius="0.05" length="0.04"/>
             </geometry>
         </collision>
